Commit message: Initial_commit

File: arm/urdf/arm2urdf.xacro (robot description, xacro)
@@ -4,4 +4,8 @@
 <xacro:include filename="$(find arm)/urdf/arm2urdf.trans" />
 <xacro:include filename="$(find arm)/urdf/arm2urdf.gazebo" />
+<xacro:include filename="$(find realsense2_description)/urdf/_d435.urdf.xacro"/>
+<xacro:sensor_d435 name="camera" topics_ns="camera" parent="wrist_2_link" publish_pointcloud="true">
+  <origin xyz="0.0 0.0215 0.01" rpy="0 0 1.5708" />
+</xacro:sensor_d435>
 <link name="base_world">
 </link>
@@ -9,6 +13,6 @@
   <inertial>
     <origin rpy="0 0 0" xyz="0 0 0"/>
-    <mass value="10"/>
-    <inertia ixx="0.0377" ixy="-0.0" ixz="0.0" iyy="0.06" iyz="0" izz="0.0376"/>
+    <mass value="100"/>
+    <inertia ixx="0.0377" ixy="0.0" ixz="0.0" iyy="0.06" iyz="0" izz="0.0376"/>
   </inertial>
   <visual>
@@ -22,5 +26,5 @@
     <origin rpy="0 0 0" xyz="0 0 0"/>
     <geometry>
-      <mesh filename="package://arm/meshes/base_link.stl" scale="0.001 0.001 0.001"/>
+      <mesh filename="package://arm/meshes/v2/base_link.stl" scale="0.001 0.001 0.001"/>
     </geometry>
   </collision>
@@ -35,5 +39,5 @@
     <origin rpy="0 0 0" xyz="0 0 -0.05"/>
     <geometry>
-      <mesh filename="package://arm/meshes/shoulder_link__4__1.stl" scale="0.001 0.001 0.001"/>
+      <mesh filename="package://arm/meshes/v2/shoulder_link__4__1.stl" scale="0.001 0.001 0.001"/>
     </geometry>
     <material name="black"/>
@@ -42,5 +46,5 @@
     <origin rpy="0 0 0" xyz="0 0 -0.05"/>
     <geometry>
-      <mesh filename="package://arm/meshes/shoulder_link__4__1.stl" scale="0.001 0.001 0.001"/>
+      <mesh filename="package://arm/meshes/v2/shoulder_link__4__1.stl" scale="0.001 0.001 0.001"/>
     </geometry>
   </collision>
@@ -48,10 +52,10 @@
 <link name="biceps_link">
   <inertial>
-    <origin rpy="0 0 0" xyz="0 0 -0.087"/>
+    <origin rpy="1.5708 0 0" xyz="0 0.087 0"/>
     <mass value="0.1569876561513581"/>
     <inertia ixx="0.002465" ixy="-3e-06" ixz="3e-06" iyy="0.000388" iyz="-0.000506" izz="0.002305"/>
   </inertial>
   <visual>
-    <origin rpy="0 0 0" xyz="0 0 -0.087"/>
+    <origin rpy="1.5708 0 0" xyz="0 0.087 0"/>
     <geometry>
       <mesh filename="package://arm/meshes/biceps_link_1.stl" scale="0.001 0.001 0.001"/>
@@ -60,5 +64,5 @@
   </visual>
   <collision>
-    <origin rpy="0 0 0" xyz="0 0 -0.087"/>
+    <origin rpy="1.5708 0 0" xyz="0 0.087 0"/>
     <geometry>
       <mesh filename="package://arm/meshes/biceps_link_1.stl" scale="0.001 0.001 0.001"/>
@@ -68,10 +72,10 @@
 <link name="forearm_link">
   <inertial>
-    <origin rpy="0 0 0" xyz="-0.05 0 -0.232"/>
+    <origin rpy="-1.5708 0 0" xyz="-0.051 -0.232 0"/>
     <mass value="0.1569876561513581"/>
     <inertia ixx="0.000327" ixy="-0.0" ixz="4e-06" iyy="0.000357" iyz="0.0" izz="7.5e-05"/>
   </inertial>
   <visual>
-    <origin rpy="0 0 0" xyz="-0.05 0 -0.232"/>
+    <origin rpy="-1.5708 0 0" xyz="-0.051 -0.232 0"/>
     <geometry>
       <mesh filename="package://arm/meshes/forearm_link_1.stl" scale="0.001 0.001 0.001"/>
@@ -80,5 +84,5 @@
   </visual>
   <collision>
-    <origin rpy="0 0 0" xyz="-0.05 0 -0.232"/>
+    <origin rpy="-1.5708 0 0" xyz="-0.051 -0.232 0"/>
     <geometry>
       <mesh filename="package://arm/meshes/forearm_link_1.stl" scale="0.001 0.001 0.001"/>
@@ -88,10 +92,10 @@
 <link name="wrist_1_link">
   <inertial>
-    <origin rpy="0 0 0" xyz="-0.2 0 -0.232"/>
+    <origin rpy="1.5708 0 0" xyz="-0.2 0.232 0"/>
     <mass value="0.14997568515174237"/>
     <inertia ixx="6.4e-05" ixy="-0.0" ixz="-0.0" iyy="5.2e-05" iyz="-9e-06" izz="4.6e-05"/>
   </inertial>
   <visual>
-    <origin rpy="0 0 0" xyz="-0.2 0 -0.232"/>
+    <origin rpy="1.5708 0 0" xyz="-0.2 0.232 0"/>
     <geometry>
       <mesh filename="package://arm/meshes/wrist_1_1.stl" scale="0.001 0.001 0.001"/>
@@ -100,5 +104,5 @@
   </visual>
   <collision>
-    <origin rpy="0 0 0" xyz="-0.2 0 -0.232"/>
+    <origin rpy="1.5708 0 0" xyz="-0.2 0.232 0"/>
     <geometry>
       <mesh filename="package://arm/meshes/wrist_1_1.stl" scale="0.001 0.001 0.001"/>
@@ -108,10 +112,10 @@
 <link name="wrist_2_link">
   <inertial>
-    <origin rpy="0 0 0" xyz="-0.28 0.0 -0.232"/>
+    <origin rpy="1.5708 1.5708 0" xyz="-0.003 0.232 -0.28"/>
     <mass value="0.12757912716999015"/>
     <inertia ixx="4.1e-05" ixy="-0.0" ixz="-0.0" iyy="2.4e-05" iyz="-1e-06" izz="3.2e-05"/>
   </inertial>
   <visual>
-    <origin rpy="0 0 0" xyz="-0.28 0.0 -0.232"/>
+    <origin rpy="1.5708 -1.5708 0" xyz="-0.003 0.232 -0.28"/>
     <geometry>
       <mesh filename="package://arm/meshes/wrist_2_1.stl" scale="0.001 0.001 0.001"/>
@@ -120,5 +124,5 @@
   </visual>
   <collision>
-    <origin rpy="0 0 0" xyz="-0.28 0.0 -0.232"/>
+    <origin rpy="1.5708 1.5708 0" xyz="-0.003 0.232 -0.28"/>
     <geometry>
       <mesh filename="package://arm/meshes/wrist_2_1.stl" scale="0.001 0.001 0.001"/>
@@ -128,17 +132,17 @@
 <link name="gripper_rail_link">
   <inertial>
-    <origin rpy="0 0 0" xyz="-0.318 0 -0.232"/>
+    <origin rpy="0 0 0" xyz="-0.32 0 -0.232"/>
     <mass value="0.02867149681670596"/>
     <inertia ixx="4e-06" ixy="-0.0" ixz="0.0" iyy="2.8e-05" iyz="0.0" izz="2.6e-05"/>
   </inertial>
   <visual>
-    <origin rpy="0 0 0" xyz="-0.318 0 -0.232"/>
+    <origin rpy="0 0 0" xyz="-0.32 0 -0.232"/>
     <geometry>
       <mesh filename="package://arm/meshes/rail_fing_supp_1.stl" scale="0.001 0.001 0.001"/>
     </geometry>
-    <material name="silver_default"/>
-  </visual>
-  <collision>
-    <origin rpy="0 0 0" xyz="-0.318 0 -0.232"/>
+    <material name="black"/>
+  </visual>
+  <collision>
+    <origin rpy="0 0 0" xyz="-0.32 0 -0.232"/>
     <geometry>
       <mesh filename="package://arm/meshes/rail_fing_supp_1.stl" scale="0.001 0.001 0.001"/>
@@ -148,17 +152,17 @@
 <link name="gripper_left_link">
   <inertial>
-    <origin rpy="0 0 0" xyz="-0.341 -0.023 -0.232"/>
+    <origin rpy="0 0 0" xyz="-0.342 -0.023 -0.232"/>
     <mass value="0.009"/>
     <inertia ixx="3e-06" ixy="0.0" ixz="0.0" iyy="3e-06" iyz="0.0" izz="1e-06"/>
   </inertial>
   <visual>
-    <origin rpy="0 0 0" xyz="-0.341 -0.023 -0.232"/>
-    <geometry>
-      <mesh filename="package://arm/meshes/finger.stl" scale="0.001 0.001 0.001"/>
-    </geometry>
-    <material name="black"/>
-  </visual>
-  <collision>
-    <origin rpy="0 0 0" xyz="-0.341 -0.023 -0.232"/>
+    <origin rpy="0 0 0" xyz="-0.342 -0.023 -0.232"/>
+    <geometry>
+      <mesh filename="package://arm/meshes/finger.stl" scale="0.001 0.001 0.001"/>
+    </geometry>
+    <material name="black"/>
+  </visual>
+  <collision>
+    <origin rpy="0 0 0" xyz="-0.342 -0.023 -0.232"/>
     <geometry>
       <mesh filename="package://arm/meshes/finger.stl" scale="0.001 0.001 0.001"/>
@@ -168,17 +172,17 @@
 <link name="gripper_right_link">
   <inertial>
-    <origin rpy="-3.1415 0 0" xyz="-0.341 0.023 0.231"/>
+    <origin rpy="-3.1415 0 0" xyz="-0.342 0.023 0.232"/>
     <mass value="0.009"/>
     <inertia ixx="3e-06" ixy="0.0" ixz="0.0" iyy="3e-06" iyz="0.0" izz="1e-06"/>
   </inertial>
   <visual>
-    <origin rpy="-3.1415 0 0" xyz="-0.341 0.023 0.231"/>
-    <geometry>
-      <mesh filename="package://arm/meshes/finger.stl" scale="0.001 0.001 0.001"/>
-    </geometry>
-    <material name="black"/>
-  </visual>
-  <collision>
-    <origin rpy="-3.1415 0 0" xyz="-0.341 0.023 0.231"/>
+    <origin rpy="-3.1415 0 0" xyz="-0.342 0.023 0.232"/>
+    <geometry>
+      <mesh filename="package://arm/meshes/finger.stl" scale="0.001 0.001 0.001"/>
+    </geometry>
+    <material name="black"/>
+  </visual>
+  <collision>
+    <origin rpy="-3.1415 0 0" xyz="-0.342 0.023 0.232"/>
     <geometry>
       <mesh filename="package://arm/meshes/finger.stl" scale="0.001 0.001 0.001"/>
@@ -198,15 +202,15 @@
 </joint>
 <joint name="joint_2" type="revolute">
-  <origin rpy="0 0 0" xyz="0 0 0.04"/>
+  <origin rpy="-1.5708 0 0" xyz="0 0 0.036"/>
   <parent link="shoulder_link"/>
   <child link="biceps_link"/>
-  <axis xyz="0.0 1.0 0.0"/>
+  <axis xyz="0 0 1"/>
   <limit effort="100" lower="-1.571" upper="1.571" velocity="1.571"/>
 </joint>
 <joint name="joint_3" type="revolute">
-  <origin rpy="0 0 0" xyz="0.05 0 0.145"/>
+  <origin rpy="0 0 0" xyz="0.051 -0.145 0"/>
   <parent link="biceps_link"/>
   <child link="forearm_link"/>
-  <axis xyz="0.0 1.0 0.0"/>
+  <axis xyz="0 0 1"/>
   <limit effort="100" lower="-1.571" upper="1.571" velocity="1.571"/>
 </joint>
@@ -215,31 +219,31 @@
   <parent link="forearm_link"/>
   <child link="wrist_1_link"/>
-  <axis xyz="0.0 1.0 0.0"/>
+  <axis xyz="0 0 1"/>
   <limit effort="100" lower="-1.745" upper="1.745" velocity="1.571"/>
 </joint>
 <joint name="joint_5" type="revolute">
-  <origin rpy="0 0 0" xyz="0.08 0 0"/>
+  <origin rpy="0 1.5708 0" xyz="0.078 0 0"/>
   <parent link="wrist_1_link"/>
   <child link="wrist_2_link"/>
-  <axis xyz="1.0 0.0 0.0"/>
+  <axis xyz="0 0 1"/>
   <limit effort="100" lower="-2.617" upper="2.617" velocity="1.571"/>
 </joint>
 <joint name="Rigid43" type="fixed">
-  <origin rpy="0 0 0" xyz="0.04 0 0"/>
+  <origin rpy="1.5708 -1.5708 0" xyz="0 0 0.043"/>
   <parent link="wrist_2_link"/>
   <child link="gripper_rail_link"/>
 </joint>
 <joint name="gripper_prismatic_joint_1" type="prismatic">
-  <origin rpy="0 0 0" xyz="0.023 0.005 0"/>
+  <origin rpy="0 0 0" xyz="0.022 0.005 0"/>
   <parent link="gripper_rail_link"/>
   <child link="gripper_left_link"/>
-  <axis xyz="0.0 1.0 0"/>
+  <axis xyz="0 1 0"/>
   <limit effort="100" lower="0" upper="0.024" velocity="0.5"/>
 </joint>
 <joint name="gripper_prismatic_joint_2" type="prismatic">
-  <origin rpy="0 0 0" xyz="0.023 -0.005 0"/>
+  <origin rpy="0 0 0" xyz="0.022 -0.005 0"/>
   <parent link="gripper_rail_link"/>
   <child link="gripper_right_link"/>
-  <axis xyz="0.0 -1.0 0"/>
+  <axis xyz="0 -1 0"/>
   <limit effort="100" lower="0" upper="0.024" velocity="0.5"/>
 </joint>
